Commit message: benchmarkt test completed

File: environments/objects/obstacle_data/duck/duck.urdf (robot description, URDF)
Before this commit: robot cube.urdf, 1 links, 0 joints
Links:
- link baseLink: geometry collision mesh filename=duck_vhacd.obj scale=3.35 3.35 3.35; visual mesh filename=duck.obj scale=3.35 3.35 3.35

Commit message: pylint inclease

File: environments/objects/obstacle_data/duck/duck.urdf (robot description, URDF)
Before this commit: robot cube.urdf, 1 links, 0 joints
Links:
- link baseLink: geometry collision mesh filename=duck_vhacd.obj scale=0.35 0.35 0.35; visual mesh filename=duck.obj scale=0.35 0.35 0.35
